File: a.kicad_sch (KiCad schematic)
At the start: 0 parts

Commit message: i2
Other:
- added sheet r (r.kicad_sch)
Changed lines of the file:
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@@
 (kicad_sch (version 20230121) (generator eeschema)
   (paper "A4")
+  (sheet (at 151.765 87.63) (size 25.4 22.225) (fields_autoplaced)
+    (stroke (width 0.1524) (type solid))
+    (fill (color 0 0 0 0.0000))
+    (property "Sheetname" "r" (at 151.765 86.9184 0)
+      (effects (font (size 1.27 1.27)) (justify left bottom))
+    )
+    (property "Sheetfile" "r.kicad_sch" (at 151.765 110.4396 0)
+      (effects (font (size 1.27 1.27)) (justify left top))
+    )
+    (instances
+      (project "a"
+        (path "/63c7d38a-b995-448a-bb92-186d24470b66" (page "2"))
+      )
+    )
+  )
   (sheet_instances
     (path "/" (page "1"))
